Commit message: test for AISR drawing space completed, ready for use

File: ws_ros2_moveit2/src/moveit_resources/panda_description/urdf/panda.urdf (robot description, URDF)
Before this commit: robot panda, 35 links, 34 joints
Joints:
- joint panda_joint8: origin xyz=0 -0.12000024 -0.325247 rpy=0 0 0 -> xyz=0 -0.10 -0.375247 rpy=0 0 0
- joint white_hand: origin xyz=0 0.12000024 0.050247 rpy=-1.57 1.57 3.14 -> xyz=0 0.10 0.100247 rpy=-1.57 1.57 3.14

Commit message: AISR model updated

File: ws_ros2_moveit2/src/moveit_resources/panda_description/urdf/panda.urdf (robot description, URDF)
Before this commit: robot panda, 35 links, 34 joints
Links:
- removed link Black_Link1
- removed link Black_Link2
- removed link Black_Link4
- removed link Black_Link5
- removed link Black_Link6
- removed link Black_Link7
- removed link Neck_Link1
- removed link Neck_Link2
- removed link Waist_Link1
- removed link Waist_Link2
- removed link base_link
- removed link black_Link3
- added link BLink1, mass 0.00330630285835291; collision mesh filename=package://moveit_resources_panda_description/meshes/l_hand/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; visual mesh filename=package://moveit_resources_panda_description/meshes/l_hand/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
- added link BLink11, mass 0.00453366979354947; collision mesh filename=package://moveit_resources_panda_description/meshes/l_hand/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; visual mesh filename=package://moveit_resources_panda_description/meshes/l_hand/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
- added link BLink111, mass 0.226288892912552; collision mesh filename=package://moveit_resources_panda_description/meshes/l_hand/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; visual mesh filename=package://moveit_resources_panda_description/meshes/l_hand/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
- added link BLink2, mass 0.00330621735666597; collision mesh filename=package://moveit_resources_panda_description/meshes/l_hand/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; visual mesh filename=package://moveit_resources_panda_description/meshes/l_hand/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
- added link BLink22, mass 0.00453367027223764; collision mesh filename=package://moveit_resources_panda_description/meshes/l_hand/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; visual mesh filename=package://moveit_resources_panda_description/meshes/l_hand/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
- added link BLink3, mass 0.00330616517571661; collision mesh filename=package://moveit_resources_panda_description/meshes/l_hand/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; visual mesh filename=package://moveit_resources_panda_description/meshes/l_hand/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
- added link BLink33, mass 0.00453366946672897; collision mesh filename=package://moveit_resources_panda_description/meshes/l_hand/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; visual mesh filename=package://moveit_resources_panda_description/meshes/l_hand/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
- added link BLink4, mass 0.00330630460851054; collision mesh filename=package://moveit_resources_panda_description/meshes/l_hand/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; visual mesh filename=package://moveit_resources_panda_description/meshes/l_hand/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
- added link BLink44, mass 0.00356888715893842; collision mesh filename=package://moveit_resources_panda_description/meshes/l_hand/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; visual mesh filename=package://moveit_resources_panda_description/meshes/l_hand/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
- added link BLink5, mass 0.00487393910083768; collision mesh filename=package://moveit_resources_panda_description/meshes/l_hand/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; visual mesh filename=package://moveit_resources_panda_description/meshes/l_hand/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
- added link BLink51, mass 0.00652741708580189; collision mesh filename=package://moveit_resources_panda_description/meshes/l_hand/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; visual mesh filename=package://moveit_resources_panda_description/meshes/l_hand/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
- added link BLink52, mass 0.00226947954597765; collision mesh filename=package://moveit_resources_panda_description/meshes/l_hand/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; visual mesh filename=package://moveit_resources_panda_description/meshes/l_hand/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
- added link BLink53, mass 0.00330869122519449; collision mesh filename=package://moveit_resources_panda_description/meshes/l_hand/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; visual mesh filename=package://moveit_resources_panda_description/meshes/l_hand/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
- added link black_link1, mass 0.154689397372487; collision mesh filename=package://moveit_resources_panda_description/meshes/black_l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; visual mesh filename=package://moveit_resources_panda_description/meshes/black_l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
- added link black_link2, mass 0.15802; collision mesh filename=package://moveit_resources_panda_description/meshes/black_l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; visual mesh filename=package://moveit_resources_panda_description/meshes/black_l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
- added link black_link3, mass 0.2616266737403; collision mesh filename=package://moveit_resources_panda_description/meshes/black_l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; visual mesh filename=package://moveit_resources_panda_description/meshes/black_l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
- added link black_link4, mass 0.14092; collision mesh filename=package://moveit_resources_panda_description/meshes/black_l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; visual mesh filename=package://moveit_resources_panda_description/meshes/black_l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
- added link black_link5, mass 0.107953940931523; collision mesh filename=package://moveit_resources_panda_description/meshes/black_l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; visual mesh filename=package://moveit_resources_panda_description/meshes/black_l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
- added link black_link6, mass 0.131069688375068; collision mesh filename=package://moveit_resources_panda_description/meshes/black_l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; visual mesh filename=package://moveit_resources_panda_description/meshes/black_l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
- added link black_link7, mass 0.025544041765819; collision mesh filename=package://moveit_resources_panda_description/meshes/black_l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; visual mesh filename=package://moveit_resources_panda_description/meshes/black_l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
- added link neck_link1, mass 0.239221970649676; collision mesh filename=package://moveit_resources_panda_description/meshes/neck_li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; visual mesh filename=package://moveit_resources_panda_description/meshes/neck_li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
- added link neck_link2, mass 1.08294216302997; collision mesh filename=package://moveit_resources_panda_description/meshes/neck_li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; visual mesh filename=package://moveit_resources_panda_description/meshes/neck_li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
- link panda_link0: mass 1.08788106388447 -> 38.318; geometry collision mesh filename=package://moveit_resources_panda_description/meshes/base_li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; visual mesh filename=package://moveit_resources_panda_description/meshes/base_li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
- link panda_link1: mass 0.46221855499898 -> 0.46222; geometry collision mesh filename=package://moveit_resources_panda_description/meshes/white_l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; visual mesh filename=package://moveit_resources_panda_description/meshes/white_l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
- link panda_link2: mass 0.103619832607522 -> 0.10361980808425; geometry collision mesh filename=package://moveit_resources_panda_description/meshes/white_l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; visual mesh filename=package://moveit_resources_panda_description/meshes/white_l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
- link panda_link3: mass 0.600118848773854 -> 0.60012; geometry collision mesh filename=package://moveit_resources_panda_description/meshes/white_l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; visual mesh filename=package://moveit_resources_panda_description/meshes/white_l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
- link panda_link4: mass 0.0620799654815404 -> 0.0620799688774293; geometry collision mesh filename=package://moveit_resources_panda_description/meshes/white_l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; visual mesh filename=package://moveit_resources_panda_description/meshes/white_l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
- link panda_link5: mass 0.439408367700066 -> 0.439407691305706; geometry collision mesh filename=package://moveit_resources_panda_description/meshes/white_l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; visual mesh filename=package://moveit_resources_panda_description/meshes/white_l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
Joints:
- removed joint dummy_joint
- removed joint waist1_joint
- removed joint waist2_joint
- removed joint waist3_joint
- added joint BLink1: type revolute, parent BLink111, child BLink1, origin xyz=0.0068852 -0.0077547 -0.08206 rpy=-1.4604 1.2485 -1.466, axis 0 0 1, limit lower=-1.6 upper=0 effort=1 velocity=1
- added joint BLink11: type revolute, parent BLink1, child BLink11, origin xyz=0.032132 0 0 rpy=-5.2101E-10 -2.8366E-11 -0.05439, axis 0 0 1, limit lower=-1.7 upper=0 effort=1 velocity=1
- added joint BLink2: type revolute, parent BLink111, child BLink2, origin xyz=-0.012436 -0.0077547 -0.082423 rpy=-1.5708 1.4093 -1.5708, axis 0 0 1, limit lower=-1.6 upper=0 effort=1 velocity=1
- added joint BLink22: type revolute, parent BLink2, child BLink22, origin xyz=0.032132 0 0 rpy=-5.0853E-10 -1.1686E-10 -0.22588, axis 0 0 1, limit lower=-1.7 upper=0 effort=1 velocity=1
- added joint BLink3: type revolute, parent BLink111, child BLink3, origin xyz=-0.031665 -0.0077547 -0.08192 rpy=-1.9857 1.4406 -1.9826, axis 0 0 1, limit lower=-1.6 upper=0 effort=1 velocity=1
- added joint BLink33: type revolute, parent BLink3, child BLink33, origin xyz=0.032132 0 0 rpy=-5.0314E-10 -1.3824E-10 -0.26815, axis 0 0 1, limit lower=-1.7 upper=0 effort=1 velocity=1
- added joint BLink4: type revolute, parent BLink111, child BLink4, origin xyz=-0.050841 -0.0077547 -0.08041 rpy=-2.0186 1.327 -2.007, axis 0 0 1, limit lower=-1.6 upper=0 effort=1 velocity=1
- added joint BLink44: type revolute, parent BLink4, child BLink44, origin xyz=0.032132 0 0 rpy=-5.1334E-10 -9.3483E-11 -0.18013, axis 0 0 1, limit lower=-1.7 upper=0 effort=1 velocity=1
- added joint BLink5: type revolute, parent BLink111, child BLink5, origin xyz=0.0010638 -0.025 -0.0059231 rpy=-1.5708 -2.455E-15 2.3555, axis 0 1 0, limit lower=-1 upper=0.3 effort=1 velocity=1
- added joint BLink51: type revolute, parent BLink5, child BLink51, origin xyz=-0.0115 -0.00075 0 rpy=-1.4988E-15 -5.5511E-17 1.8988, axis 0 0 -1, limit lower=0 upper=0.4 effort=1 velocity=1
- added joint BLink52: type revolute, parent BLink51, child BLink52, origin xyz=0.056001 0 0 rpy=-1.3323E-15 -2.7756E-17 -3.0416, axis 0 0 1, limit lower=-0.4 upper=0 effort=1 velocity=1
- added joint BLink53: type revolute, parent BLink52, child BLink53, origin xyz=-0.022653 0 0 rpy=1.2712E-14 -9.7145E-17 2.856, axis 0 0 1, limit lower=-1 upper=0 effort=1 velocity=1
- added joint black_hand: type fixed, parent black_link7, child BLink111, origin xyz=0.1 -0.02 -0.02 rpy=-1.5707963267949 3.14159265358956 1.5707963267949
- added joint fixed: type fixed, parent dummy_link, child panda_link0, origin xyz=0 0 0 rpy=0 0 1.5708
- joint Link11: limit lower=-1.7 upper=0 effort=1 velocity=100 -> lower=-1.7 upper=0 effort=1 velocity=1; type fixed -> revolute
- joint Link22: limit lower=-1.7 upper=0 effort=1 velocity=100 -> lower=-1.7 upper=0 effort=1 velocity=1; type fixed -> revolute
- joint Link3: limit lower=-1.6 upper=0 effort=1 velocity=100 -> lower=-1.6 upper=0 effort=1 velocity=1; type fixed -> revolute
- joint Link33: limit lower=-1.7 upper=0 effort=1 velocity=100 -> lower=-1.7 upper=0 effort=1 velocity=1; type fixed -> revolute
- joint Link4: limit lower=-1.6 upper=0 effort=1 velocity=100 -> lower=-1.6 upper=0 effort=1 velocity=1; type fixed -> revolute
- joint Link44: limit lower=-1.7 upper=0 effort=1 velocity=100 -> lower=-1.7 upper=0 effort=1 velocity=1; type fixed -> revolute
- joint Link5: limit lower=-1 upper=0.3 effort=1 velocity=100 -> lower=-1 upper=0.3 effort=1 velocity=1; type fixed -> revolute
- joint Link51: limit lower=0 upper=0.4 effort=1 velocity=100 -> lower=0 upper=0.4 effort=1 velocity=1; type fixed -> revolute
- joint Link52: limit lower=-0.4 upper=0 effort=1 velocity=100 -> lower=-0.4 upper=0 effort=1 velocity=1; type fixed -> revolute
- joint Link53: limit lower=-1 upper=0 effort=1 velocity=100 -> lower=-1 upper=0 effort=1 velocity=1; type fixed -> revolute
- joint black1_joint: axis 0 0 -1 -> 0 0 1; child Black_Link1 -> black_link1; limit lower=-2.0 upper=0.0 effort=100.0 velocity=100.0 -> lower=-1.57 upper=2.3 effort=0 velocity=0; origin xyz=-0.13313 -0.14666 -0.0002 rpy=-1.5708 0 -1.309 -> xyz=0.133825302830738 0 1.15071708300629 rpy=-3.14159265358635 1.30899693899575 0
- joint black2_joint: axis 0 0 -1 -> 0 0 1; child Black_Link2 -> black_link2; limit lower=0.0 upper=1.5 effort=100.0 velocity=100.0 -> lower=-2.3 upper=0.6 effort=0 velocity=0; origin xyz=0 0 -0.1165 rpy=-1.5708 -1.309 0 -> xyz=0 0 -0.116500000000004 rpy=1.5707963267949 1.30899693899575 0; parent Black_Link1 -> black_link1
- joint black3_joint: child black_Link3 -> black_link3; limit lower=-1.5 upper=1.5 effort=100.0 velocity=100.0 -> lower=-2.7 upper=0 effort=0 velocity=0; origin xyz=0 -0.11415 -0.0002 rpy=-1.5708 0 0 -> xyz=0.0255223354162147 0.111465388775543 0 rpy=1.5707963267949 0 -0.22509081564678; parent Black_Link2 -> black_link2
- joint black4_joint: axis 0 0 1 -> 0 0 -1; child Black_Link4 -> black_link4; limit lower=0.0 upper=2.0 effort=100.0 velocity=100.0 -> lower=-1.8 upper=0.0 effort=0 velocity=0; origin xyz=0 0 -0.1482 rpy=1.5708 0 1.5708 -> xyz=0 0 -0.148 rpy=-1.57079632679489 0.22509081564678 0; parent black_Link3 -> black_link3
- joint black5_joint: child Black_Link5 -> black_link5; limit lower=-1.5 upper=1.5 effort=100.0 velocity=100.0 -> lower=-3.0 upper=3.0 effort=0 velocity=0; origin xyz=0 -0.10775 0 rpy=-1.5708 -1.5708 0 -> xyz=0.0240715686458765 0.10512935880584 0 rpy=1.57079632679489 0 -0.22509081564678; parent Black_Link4 -> black_link4
- joint black6_joint: axis 0 0 1 -> 0 0 -1; child Black_Link6 -> black_link6; limit lower=-1.5 upper=1.5 effort=100.0 velocity=100.0 -> lower=-0.2 upper=0.2 effort=0 velocity=0; origin xyz=0 0 -0.0481 rpy=1.5708 0 0 -> xyz=0 0 -0.0480000000000004 rpy=-1.57079632679489 0.22509081564678 0; parent Black_Link5 -> black_link5
- joint black7_joint: child Black_Link7 -> black_link7; limit lower=-1.5 upper=1.5 effort=100.0 velocity=100.0 -> lower=-0.2 upper=0.2 effort=0 velocity=0; origin xyz=0 -0.078 0 rpy=0 1.5708 0 -> xyz=0.0442154818872393 0.0698945002234028 0.000100000000135983 rpy=1.57079632679467 0 1.34570551114812; parent Black_Link6 -> black_link6
- joint neck1_joint: child Neck_Link1 -> neck_link1; limit lower=-1.5 upper=1.5 effort=100.0 velocity=100.0 -> lower=-1.57 upper=1.57 effort=0 velocity=0; origin xyz=0.0005 -0.22275 -0.0002 rpy=1.5708 0 0 -> xyz=0 0 1.22674746798424 rpy=0 0 0
- joint neck2_joint: child Neck_Link2 -> neck_link2; limit lower=-0.5 upper=0.5 effort=100.0 velocity=100.0 -> lower=-0.5 upper=0.5 effort=0 velocity=0; origin xyz=0.0002 0 0.0415 rpy=1.5708 0 1.5708 -> xyz=0 0 0.0415000000000025 rpy=-1.5707963267949 0 -1.55367583356864; parent Neck_Link1 -> neck_link1
- joint panda_finger_joint1: limit lower=-1.6 upper=0 effort=1 velocity=100 -> lower=-1.6 upper=0 effort=1 velocity=1; type fixed -> revolute
- joint panda_finger_joint2: limit lower=-1.6 upper=0 effort=1 velocity=100 -> lower=-1.6 upper=0 effort=1 velocity=1; type fixed -> revolute
- joint panda_joint1: limit lower=0.0 upper=2.0 effort=100.0 velocity=100.0 -> lower=-1.57 upper=2.3 effort=0 velocity=0; origin xyz=0.20962 -0.16689 -0.0002 rpy=1.5708 0 1.309 -> xyz=-0.209119220989971 0 1.17089202757203 rpy=0 -1.30899693899575 0
- joint panda_joint2: axis 0 0 1 -> 0 0 -1; limit lower=0.0 upper=1.5 effort=100.0 velocity=100.0 -> lower=-2.3 upper=0 effort=0 velocity=0; origin xyz=0 0 0.055 rpy=1.5708 -1.5708 0 -> xyz=0 0 0.0549999999999993 rpy=-1.5707963267949 1.30899693899575 0
- joint panda_joint3: limit lower=-1.5 upper=1.5 effort=100.0 velocity=100.0 -> lower=0.00 upper=2.57 effort=0 velocity=0; origin xyz=0 -0.08 0.0045 rpy=-1.5708 0 0 -> xyz=-0.0167788293984912 0.0782206550982036 -0.00450000000001032 rpy=1.57079632679491 1.56 0.211304299584282
- joint panda_joint4: limit lower=0.0 upper=2.0 effort=100.0 velocity=100.0 -> lower=-2.0 upper=0.0 effort=0 velocity=0; origin xyz=0 0 -0.163 rpy=1.5708 0 1.5708 -> xyz=0 0 -0.163 rpy=1.57079632679491 0.211304299584282 3.14159265358956
- joint panda_joint5: axis 0 0 -1 -> 0 0 1; limit lower=-1.5 upper=1.5 effort=100.0 velocity=100.0 -> lower=-3.0 upper=3.0 effort=0 velocity=0; origin xyz=0 -0.06 0 rpy=-1.5708 -1.5708 0 -> xyz=0.0125841220490822 -0.0586654913237358 0 rpy=1.57079632679491 -1.51 -2.93028835400551
- joint panda_joint8: origin xyz=0 -0.10 -0.375247 rpy=0 0 0 -> xyz=0.03 0.075 -0.373 rpy=0 0 0
- joint white_hand: axis -1 0 0 -> (none); limit lower=-3.14 upper=3.14 effort=100.0 velocity=100.0 -> (none); origin xyz=0 0.10 0.100247 rpy=-1.57 1.57 3.14 -> xyz=-0.01 -0.02 -0.28 rpy=-1.5707963267948966 1.57 0; parent panda_link8 -> panda_link7; type revolute -> fixed

Commit message: moveit with pub/sub achieved, logic of lifting the pen added, AISR can write now

File: ws_ros2_moveit2/src/moveit_resources/panda_description/urdf/panda.urdf (robot description, URDF)
Before this commit: robot panda, 45 links, 44 joints
Joints:
- joint panda_joint2: limit lower=-2.3 upper=0 effort=0 velocity=0 -> lower=-2.0 upper=0.15 effort=0 velocity=0
- joint panda_joint3: limit lower=0.00 upper=2.57 effort=0 velocity=0 -> lower=-1.57 upper=1.0 effort=0 velocity=0
